File: Hardware/PCB&Eletronic/TCC_Flow.kicad_sch (KiCad schematic)
At the start: 41 parts, among them Q1 BC337, Q2 BC337, Q3 BC337, Q4 BC337

Commit message: [PCB] Add updated pcb and Doc
Parts:
- removed C5: 1uF, Capacitor_THT:CP_Radial_D5.0mm_P2.00mm, symbol Device:C
- removed R1, R2: 4.6K, Resistor_THT:R_Axial_DIN0204_L3.6mm_D1.6mm_P5.08mm_Vertical, symbol Device:R
- removed R7: 220, Resistor_THT:R_Axial_DIN0204_L3.6mm_D1.6mm_P5.08mm_Vertical, symbol Device:R
- added C9: 1uF, Capacitor_THT:CP_Radial_D5.0mm_P2.00mm, symbol Device:C
- added R10, R9: 4.7K, Resistor_THT:R_Axial_DIN0204_L3.6mm_D1.6mm_P5.08mm_Horizontal, symbol Device:R
- added R11: 220, Resistor_THT:R_Axial_DIN0204_L3.6mm_D1.6mm_P5.08mm_Horizontal, symbol Device:R
- Clock1: footprint Connector_Wire:SolderWire-0.1sqmm_1x05_P3.6mm_D0.4mm_OD1mm -> Connector_PinHeader_2.54mm:PinHeader_1x05_P2.54mm_Horizontal
- MicroSd1: footprint Connector_Wire:SolderWire-0.1sqmm_1x06_P3.6mm_D0.4mm_OD1mm -> Connector_PinHeader_2.54mm:PinHeader_1x06_P2.54mm_Horizontal
- Pirani1: footprint Connector_RJ:RJ45_Amphenol_RJHSE5380 -> Connector_RJ:RJ45_Wuerth_7499010001A_Horizontal
- PwSpp15V1: footprint Connector_BarrelJack:BarrelJack_Horizontal -> Connector_PinHeader_2.54mm:PinHeader_1x02_P2.54mm_Vertical
- PwSpp15V2, PwSpp5V1: footprint Connector_Wire:SolderWire-0.1sqmm_1x02_P3.6mm_D0.4mm_OD1mm -> Connector_PinHeader_2.54mm:PinHeader_1x02_P2.54mm_Vertical
- Q1, Q2, Q3, Q4: footprint Package_TO_SOT_THT:TO-92_Inline -> Package_TO_SOT_THT:TO-92L_Inline_Wide
- R1: renamed from R3; value 500 -> 470; footprint Resistor_THT:R_Axial_DIN0204_L3.6mm_D1.6mm_P5.08mm_Vertical -> Resistor_THT:R_Axial_DIN0204_L3.6mm_D1.6mm_P5.08mm_Horizontal
- R12: renamed from R8; footprint Resistor_THT:R_Axial_DIN0204_L3.6mm_D1.6mm_P5.08mm_Vertical -> Resistor_THT:R_Axial_DIN0204_L3.6mm_D1.6mm_P5.08mm_Horizontal
- R13: renamed from R11; footprint Resistor_THT:R_Axial_DIN0204_L3.6mm_D1.6mm_P5.08mm_Vertical -> Resistor_THT:R_Axial_DIN0204_L3.6mm_D1.6mm_P5.08mm_Horizontal
- R14: renamed from R10; footprint Resistor_THT:R_Axial_DIN0204_L3.6mm_D1.6mm_P5.08mm_Vertical -> Resistor_THT:R_Axial_DIN0204_L3.6mm_D1.6mm_P5.08mm_Horizontal
- R15: renamed from R12; footprint Resistor_THT:R_Axial_DIN0204_L3.6mm_D1.6mm_P5.08mm_Vertical -> Resistor_THT:R_Axial_DIN0204_L3.6mm_D1.6mm_P5.08mm_Horizontal
- R2: renamed from R9; value 500 -> 470; footprint Resistor_THT:R_Axial_DIN0204_L3.6mm_D1.6mm_P5.08mm_Vertical -> Resistor_THT:R_Axial_DIN0204_L3.6mm_D1.6mm_P5.08mm_Horizontal
- R3: renamed from R4; value 500 -> 470; footprint Resistor_THT:R_Axial_DIN0204_L3.6mm_D1.6mm_P5.08mm_Vertical -> Resistor_THT:R_Axial_DIN0204_L3.6mm_D1.6mm_P5.08mm_Horizontal
- R4: renamed from R15; value 500 -> 470; footprint Resistor_THT:R_Axial_DIN0204_L3.6mm_D1.6mm_P5.08mm_Vertical -> Resistor_THT:R_Axial_DIN0204_L3.6mm_D1.6mm_P5.08mm_Horizontal
- R5: value 500 -> 470; footprint Resistor_THT:R_Axial_DIN0204_L3.6mm_D1.6mm_P5.08mm_Vertical -> Resistor_THT:R_Axial_DIN0204_L3.6mm_D1.6mm_P5.08mm_Horizontal
- R6: renamed from R14; value 500 -> 470; footprint Resistor_THT:R_Axial_DIN0204_L3.6mm_D1.6mm_P5.08mm_Vertical -> Resistor_THT:R_Axial_DIN0204_L3.6mm_D1.6mm_P5.08mm_Horizontal
- R7: renamed from R6; value 500 -> 470; footprint Resistor_THT:R_Axial_DIN0204_L3.6mm_D1.6mm_P5.08mm_Vertical -> Resistor_THT:R_Axial_DIN0204_L3.6mm_D1.6mm_P5.08mm_Horizontal
- R8: renamed from R13; value 500 -> 470; footprint Resistor_THT:R_Axial_DIN0204_L3.6mm_D1.6mm_P5.08mm_Vertical -> Resistor_THT:R_Axial_DIN0204_L3.6mm_D1.6mm_P5.08mm_Horizontal
- Tela1: footprint Connector_Wire:SolderWire-0.1sqmm_1x04_P3.6mm_D0.4mm_OD1mm -> Connector_Wire:SolderWire-0.5sqmm_1x04_P4.6mm_D0.9mm_OD2.1mm
- U1: value (none) -> ESP-01v090; footprint (none) -> esp:ESP-01
- renumbered C6 to C2, C8 to C3, C2 to C4, C3 to C5, C9 to C6, C4 to C8
Connections:
- net at XA1.A5: now also R10.1, R9.1
- net at Clock1.2 (Pin_2), MicroSd1.1 (Pin_1), PwSpp15V1.2 (Pin_2)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: now also C1.2, C2.2, C3.2, C4.2, C5.2, C6.2, C7.2, C8.2, MFC1.4 (Pin_4), MFC1.7 (Pin_7), MFC2.4 (Pin_4), MFC2.7 (Pin_7), MFC3.4 (Pin_4), MFC3.7 (Pin_7), MFC4.4 (Pin_4), MFC4.7 (Pin_7), Pirani1.4 (Pin_4), Pirani1.7 (Pin_7), Q1.3 (E), Q2.3 (E), Q3.3 (E), Q4.3 (E), Tela1.1 (Pin_1), U1.2 (GND), C9.2, R9.2
- net at MFC1.3 (Pin_3), MFC2.3 (Pin_3), MFC3.3 (Pin_3)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: now also Pirani1.8 (Pin_8); no longer Pirani1.1 (Pin_1)
- net at Pirani1.6 (Pin_6): now also R11.1
- removed net GND: C1.2, C2.2, C3.2, C4.2, C5.2, C6.2, C7.2, C8.2, MFC1.4 (Pin_4), MFC1.7 (Pin_7), MFC2.4 (Pin_4), MFC2.7 (Pin_7), MFC3.4 (Pin_4), MFC3.7 (Pin_7), MFC4.4 (Pin_4), MFC4.7 (Pin_7), Pirani1.2 (Pin_2), Pirani1.5 (Pin_5), Q1.3 (E), Q2.3 (E), Q3.3 (E), Q4.3 (E), Tela1.1 (Pin_1), U1.2 (GND)
- new net: C9.1, R10.2, R11.2
